Commit message: add inertia calculation script

File: config/my_mobile_robot_with_hand.urdf (robot description, URDF)
Before this commit: robot my_mobile_robot, 8 links, 7 joints
Links:
- added link center_wheel, mass 0.1; collision cylinder length=0.05 radius=0.05; visual cylinder length=0.05 radius=0.05
- link base_link: geometry collision box size=0.5 0.3 0.23; visual box size=0.5 0.3 0.23
- link hand_base_link: geometry collision box size=0.06 0.5 0.15; visual box size=0.06 0.5 0.15
- link hand_left: geometry collision box size=0.1 0.05 0.3; visual box size=0.1 0.05 0.3
- link hand_right: geometry collision box size=0.1 0.05 0.3; visual box size=0.1 0.05 0.3
- link left_wheel: geometry collision cylinder length=0.05 radius=0.05; visual cylinder length=0.05 radius=0.05
Joints:
- added joint center_wheel_joint: type fixed, parent base_link, child center_wheel, origin xyz=0.2 0 -0.09 rpy=1.57 0 0
- joint left_wheel_joint: origin xyz=0.0 0.125 -.09 rpy=-1.5708 0 0 -> xyz=-0.2 0.125 -.09 rpy=-1.5708 0 0
- joint right_wheel_joint: origin xyz=0.0 -0.125 -.09 rpy=-1.5708 0 0 -> xyz=-0.2 -0.125 -.09 rpy=-1.5708 0 0
